File: DB9-rj45-breakout.kicad_pcb (KiCad board)
At the start: 2 copper layers, 32 x 33 mm, 4 parts, among them CN1 1x9, CN2 1x8

Commit message: b toggle conf
Changed lines of the file:
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@@
     (visible_elements FFFFFF7F)
     (pcbplotparams
-      (layerselection 0x010fc_ffffffff)
+      (layerselection 0x010f0_ffffffff)
       (usegerberextensions false)
       (usegerberattributes false)
@@
       (outputformat 1)
       (mirror false)
-      (drillshape 1)
+      (drillshape 0)
       (scaleselection 1)
-      (outputdirectory ""))
+      (outputdirectory "output/"))
   )
   (net 0 "")
@@
     (add_net /up)
     (add_net "Net-(CN1-Pad5)")
+  )
+  (module modular-jack:RJHSE-5080 (layer F.Cu)
+    (at 150 125)
+    (fp_text reference CN2 (at 0 0.5) (layer F.Fab)
+      (effects (font (size 1 1) (thickness 0.15)))
+    )
+    (fp_text value 1x8 (at 0 -0.5) (layer F.Fab) hide
+      (effects (font (size 1 1) (thickness 0.15)))
+    )
+    (fp_line (start -8 -10) (end -8 4.8) (layer F.SilkS) (width 0.12))
+    (fp_line (start 8 -10) (end 8 4.8) (layer F.SilkS) (width 0.12))
+    (fp_line (start -8 -10) (end 8 -10) (layer F.SilkS) (width 0.12))
+    (fp_line (start 7.875 5.08) (end 7.87 -9.91) (layer Dwgs.User) (width 0.12))
+    (fp_line (start -7.875 -9.91) (end -7.875 5.08) (layer Dwgs.User) (width 0.12))
+    (fp_line (start -7.875 -9.91) (end 7.87 -9.91) (layer Dwgs.User) (width 0.12))
+    (fp_line (start -7.875 5.08) (end 7.875 5.08) (layer Dwgs.User) (width 0.12))
+    (pad "" np_thru_hole circle (at -6.35 0 90) (size 3.25 3.25) (drill 3.25) (layers *.Cu *.Mask))
+    (pad "" np_thru_hole circle (at 6.35 0 90) (size 3.25 3.25) (drill 3.25) (layers *.Cu *.Mask))
+    (pad 8 thru_hole circle (at -3.555 -4.32) (size 1.5 1.5) (drill 0.89) (layers *.Cu *.Mask)
+      (net 7 /5V))
+    (pad 7 thru_hole circle (at -2.54 -2.54) (size 1.5 1.5) (drill 0.89) (layers *.Cu *.Mask)
+      (net 9 /b))
+    (pad 6 thru_hole circle (at -1.525 -4.32) (size 1.5 1.5) (drill 0.89) (layers *.Cu *.Mask)
+      (net 6 /a))
+    (pad 5 thru_hole circle (at -0.51 -2.54) (size 1.5 1.5) (drill 0.89) (layers *.Cu *.Mask)
+      (net 5 /right))
+    (pad 4 thru_hole circle (at 0.505 -4.32) (size 1.5 1.5) (drill 0.89) (layers *.Cu *.Mask)
+      (net 4 /left))
+    (pad 3 thru_hole circle (at 1.52 -2.54) (size 1.5 1.5) (drill 0.89) (layers *.Cu *.Mask)
+      (net 3 /down))
+    (pad 2 thru_hole circle (at 2.535 -4.32) (size 1.5 1.5) (drill 0.89) (layers *.Cu *.Mask)
+      (net 2 /up))
+    (pad 1 thru_hole circle (at 3.55 -2.54) (size 1.5 1.5) (drill 0.89) (layers *.Cu *.Mask)
+      (net 8 /GND))
+    (model ${KICAD_SYMBOL_DIR}/3d/M-RJHSE-5080-REVT1.STEP
+      (offset (xyz 0 1 3))
+      (scale (xyz 1 1 1))
+      (rotate (xyz -90 0 0))
+    )
   )
   (module PCB:M3 (layer F.Cu)
@@
     (model "${KICAD_SYMBOL_DIR}/3d/DB9 - 203-09SCKKBE.STEP"
       (offset (xyz 0 -9.1 6.5))
-      (scale (xyz 1 1 1))
-      (rotate (xyz -90 0 0))
-    )
-  )
-  (module modular-jack:RJHSE-5080 (layer F.Cu)
-    (at 150 125)
-    (fp_text reference CN2 (at 0 0.5) (layer F.SilkS)
-      (effects (font (size 1 1) (thickness 0.15)))
-    )
-    (fp_text value 1x8 (at 0 -0.5) (layer F.Fab)
-      (effects (font (size 1 1) (thickness 0.15)))
-    )
-    (fp_line (start -7.875 5.08) (end 7.875 5.08) (layer Dwgs.User) (width 0.12))
-    (fp_line (start -7.875 -9.91) (end 7.87 -9.91) (layer Dwgs.User) (width 0.12))
-    (fp_line (start -7.875 -9.91) (end -7.875 5.08) (layer Dwgs.User) (width 0.12))
-    (fp_line (start 7.875 5.08) (end 7.87 -9.91) (layer Dwgs.User) (width 0.12))
-    (fp_line (start -8 -10) (end 8 -10) (layer F.SilkS) (width 0.12))
-    (fp_line (start 8 -10) (end 8 4.8) (layer F.SilkS) (width 0.12))
-    (fp_line (start -8 -10) (end -8 4.8) (layer F.SilkS) (width 0.12))
-    (pad 1 thru_hole circle (at 3.55 -2.54) (size 1.5 1.5) (drill 0.89) (layers *.Cu *.Mask)
-      (net 8 /GND))
-    (pad 2 thru_hole circle (at 2.535 -4.32) (size 1.5 1.5) (drill 0.89) (layers *.Cu *.Mask)
-      (net 2 /up))
-    (pad 3 thru_hole circle (at 1.52 -2.54) (size 1.5 1.5) (drill 0.89) (layers *.Cu *.Mask)
-      (net 3 /down))
-    (pad 4 thru_hole circle (at 0.505 -4.32) (size 1.5 1.5) (drill 0.89) (layers *.Cu *.Mask)
-      (net 4 /left))
-    (pad 5 thru_hole circle (at -0.51 -2.54) (size 1.5 1.5) (drill 0.89) (layers *.Cu *.Mask)
-      (net 5 /right))
-    (pad 6 thru_hole circle (at -1.525 -4.32) (size 1.5 1.5) (drill 0.89) (layers *.Cu *.Mask)
-      (net 6 /a))
-    (pad 7 thru_hole circle (at -2.54 -2.54) (size 1.5 1.5) (drill 0.89) (layers *.Cu *.Mask)
-      (net 9 /b))
-    (pad 8 thru_hole circle (at -3.555 -4.32) (size 1.5 1.5) (drill 0.89) (layers *.Cu *.Mask)
-      (net 7 /5V))
-    (pad "" np_thru_hole circle (at 6.085 0 90) (size 3.25 3.25) (drill 3.25) (layers *.Cu *.Mask))
-    (pad "" np_thru_hole circle (at -6.085 0 90) (size 3.25 3.25) (drill 3.25) (layers *.Cu *.Mask))
-    (model ${KICAD_SYMBOL_DIR}/3d/M-RJHSE-5080-REVT1.STEP
-      (offset (xyz 0 1 3))
       (scale (xyz 1 1 1))
       (rotate (xyz -90 0 0))
@@
     (polygon
       (pts
-        (xy 166 128) (xy 134 128) (xy 134 93) (xy 166 93)
+        (xy 166 127) (xy 134 127) (xy 134 94) (xy 166 94)
       )
     )
@@
     (polygon
       (pts
-        (xy 166 128) (xy 134 128) (xy 134 93) (xy 166 93)
+        (xy 166 127) (xy 134 127) (xy 134 94) (xy 166 94)
       )
     )

Commit message: added toggle switch to select up button
Parts:
- added SW1: spdt, switch:100SP1T1B4M2QE, F.Cu at (150.0, 110.5)
Connections:
- CN2 pad 2: /up -> Net-(CN2-Pad2)
Routing:
- net Net-(CN2-Pad2): track 0.00 -> 11.1 mm
- net /up: track 20.0 -> 10.9 mm
- net /right: track 26.4 -> 28.9 mm
- net /left: track 19.0 -> 21.0 mm
- net /down: track 25.9 -> 27.8 mm
- net /a: track 25.9 -> 25.1 mm
Changed lines of the file:
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@@
     (thickness 1.6)
     (drawings 7)
-    (tracks 32)
+    (tracks 43)
     (zones 0)
-    (modules 4)
-    (nets 10)
+    (modules 5)
+    (nets 11)
   )
   (page A4)
@@
   (net 8 /GND)
   (net 9 /b)
+  (net 10 "Net-(CN2-Pad2)")
   (net_class Default "This is the default net class."
     (clearance 0.2)
@@
     (add_net /up)
     (add_net "Net-(CN1-Pad5)")
+    (add_net "Net-(CN2-Pad2)")
+  )
+  (module switch:100SP1T1B4M2QE (layer F.Cu)
+    (at 150 110.5)
+    (fp_text reference SW1 (at 0 0) (layer F.Fab) hide
+      (effects (font (size 0.5 0.5) (thickness 0.125)))
+    )
+    (fp_text value spdt (at 0 -0.5) (layer F.Fab) hide
+      (effects (font (size 1 1) (thickness 0.15)))
+    )
+    (fp_line (start -6.35 -3.43) (end 6.35 -3.43) (layer F.Fab) (width 0.12))
+    (fp_line (start -6.35 3.43) (end 6.35 3.43) (layer F.Fab) (width 0.12))
+    (fp_line (start 6.35 3.43) (end 6.35 -3.43) (layer F.Fab) (width 0.12))
+    (fp_line (start -6.35 3.43) (end -6.35 -3.43) (layer F.Fab) (width 0.12))
+    (pad 1 thru_hole circle (at -4.7 0) (size 3 3) (drill 1.85) (layers *.Cu *.Mask)
+      (net 9 /b))
+    (pad 2 thru_hole circle (at 0 0) (size 3 3) (drill 1.85) (layers *.Cu *.Mask)
+      (net 2 /up))
+    (pad 3 thru_hole circle (at 4.7 0) (size 3 3) (drill 1.85) (layers *.Cu *.Mask)
+      (net 10 "Net-(CN2-Pad2)"))
+    (model ${KICAD_SYMBOL_DIR}/3d/e-switch/100SPxT1B4M2xE.stp
+      (offset (xyz 0 0 -24))
+      (scale (xyz 0.9 1 1))
+      (rotate (xyz 0 0 0))
+    )
   )
   (module modular-jack:RJHSE-5080 (layer F.Cu)
@@
       (net 3 /down))
     (pad 2 thru_hole circle (at 2.535 -4.32) (size 1.5 1.5) (drill 0.89) (layers *.Cu *.Mask)
-      (net 2 /up))
+      (net 10 "Net-(CN2-Pad2)"))
     (pad 1 thru_hole circle (at 3.55 -2.54) (size 1.5 1.5) (drill 0.89) (layers *.Cu *.Mask)
       (net 8 /GND))
@@
   (gr_line (start 166 94) (end 166 122) (layer Edge.Cuts) (width 0.05))
   (gr_line (start 134 94) (end 166 94) (layer Edge.Cuts) (width 0.05))
-  (segment (start 155.54 101.92) (end 152.535 104.925) (width 0.5) (layer B.Cu) (net 2))
-  (segment (start 152.535 104.925) (end 152.535 120.68) (width 0.5) (layer B.Cu) (net 2))
-  (segment (start 152.720001 123.660001) (end 154.126001 123.660001) (width 0.5) (layer F.Cu) (net 3))
-  (segment (start 152.77 118.67) (end 152.77 101.92) (width 0.5) (layer F.Cu) (net 3))
-  (segment (start 154.750001 120.650001) (end 152.77 118.67) (width 0.5) (layer F.Cu) (net 3))
-  (segment (start 154.126001 123.660001) (end 154.750001 123.036001) (width 0.5) (layer F.Cu) (net 3))
-  (segment (start 151.52 122.46) (end 152.720001 123.660001) (width 0.5) (layer F.Cu) (net 3))
-  (segment (start 154.750001 123.036001) (end 154.750001 120.650001) (width 0.5) (layer F.Cu) (net 3))
-  (segment (start 150.505 120.68) (end 150 120.175) (width 0.5) (layer F.Cu) (net 4))
-  (segment (start 150 120.175) (end 150 101.92) (width 0.5) (layer F.Cu) (net 4))
-  (segment (start 147.23 101.92) (end 147.23 117.67) (width 0.5) (layer F.Cu) (net 5))
-  (segment (start 145.244999 119.655001) (end 145.244999 122.144999) (width 0.5) (layer F.Cu) (net 5))
-  (segment (start 147.23 117.67) (end 145.244999 119.655001) (width 0.5) (layer F.Cu) (net 5))
-  (segment (start 148.740001 123.209999) (end 149.49 122.46) (width 0.5) (layer F.Cu) (net 5))
-  (segment (start 148.289999 123.660001) (end 148.740001 123.209999) (width 0.5) (layer F.Cu) (net 5))
-  (segment (start 146.760001 123.660001) (end 148.289999 123.660001) (width 0.5) (layer F.Cu) (net 5))
-  (segment (start 145.244999 122.144999) (end 146.760001 123.660001) (width 0.5) (layer F.Cu) (net 5))
-  (segment (start 153.305001 99.929999) (end 154.155 99.08) (width 0.5) (layer F.Cu) (net 6))
-  (segment (start 152.735 100.5) (end 153.305001 99.929999) (width 0.5) (layer F.Cu) (net 6))
-  (segment (start 149.495998 100.5) (end 152.735 100.5) (width 0.5) (layer F.Cu) (net 6))
-  (segment (start 148.625 120.53) (end 148.625 101.370998) (width 0.5) (layer F.Cu) (net 6))
-  (segment (start 148.625 101.370998) (end 149.495998 100.5) (width 0.5) (layer F.Cu) (net 6))
-  (segment (start 148.475 120.68) (end 148.625 120.53) (width 0.5) (layer F.Cu) (net 6))
-  (segment (start 146.445 108.055) (end 146.445 120.68) (width 0.5) (layer B.Cu) (net 7))
-  (segment (start 151.385 103.115) (end 146.445 108.055) (width 0.5) (layer B.Cu) (net 7))
-  (segment (start 151.385 99.08) (end 151.385 103.115) (width 0.5) (layer B.Cu) (net 7))
-  (segment (start 145.845 100.282081) (end 145.845 99.08) (width 0.5) (layer B.Cu) (net 9))
-  (segment (start 145.845 103.407508) (end 145.845 100.282081) (width 0.5) (layer B.Cu) (net 9))
-  (segment (start 145.244999 104.007509) (end 145.845 103.407508) (width 0.5) (layer B.Cu) (net 9))
-  (segment (start 145.244999 121.305659) (end 145.244999 104.007509) (width 0.5) (layer B.Cu) (net 9))
-  (segment (start 146.39934 122.46) (end 145.244999 121.305659) (width 0.5) (layer B.Cu) (net 9))
-  (segment (start 147.46 122.46) (end 146.39934 122.46) (width 0.5) (layer B.Cu) (net 9))
+  (segment (start 155.54 104.96) (end 155.54 101.92) (width 0.5) (layer F.Cu) (net 2))
+  (segment (start 150 110.5) (end 155.54 104.96) (width 0.5) (layer F.Cu) (net 2))
+  (segment (start 157 120.786002) (end 157 106.15) (width 0.5) (layer B.Cu) (net 3))
+  (segment (start 154.126001 123.660001) (end 157 120.786002) (width 0.5) (layer B.Cu) (net 3))
+  (segment (start 152.740001 123.660001) (end 154.126001 123.660001) (width 0.5) (layer B.Cu) (net 3))
+  (segment (start 157 106.15) (end 153.619999 102.769999) (width 0.5) (layer B.Cu) (net 3))
+  (segment (start 151.54 122.46) (end 152.740001 123.660001) (width 0.5) (layer B.Cu) (net 3))
+  (segment (start 153.619999 102.769999) (end 152.77 101.92) (width 0.5) (layer B.Cu) (net 3))
+  (segment (start 151.52 122.46) (end 151.54 122.46) (width 0.5) (layer B.Cu) (net 3))
+  (segment (start 150 104.5) (end 150 101.92) (width 0.5) (layer F.Cu) (net 4))
+  (segment (start 147.5 107) (end 150 104.5) (width 0.5) (layer F.Cu) (net 4))
+  (segment (start 147.5 116.61434) (end 147.5 107) (width 0.5) (layer F.Cu) (net 4))
+  (segment (start 150.505 119.61934) (end 147.5 116.61434) (width 0.5) (layer F.Cu) (net 4))
+  (segment (start 150.505 120.68) (end 150.505 119.61934) (width 0.5) (layer F.Cu) (net 4))
+  (segment (start 147.23 101.92) (end 147.23 104.27) (width 0.5) (layer B.Cu) (net 5))
+  (segment (start 143.349999 108.150001) (end 143.349999 121.349999) (width 0.5) (layer B.Cu) (net 5))
+  (segment (start 147.23 104.27) (end 143.349999 108.150001) (width 0.5) (layer B.Cu) (net 5))
+  (segment (start 143.349999 121.349999) (end 146 124) (width 0.5) (layer B.Cu) (net 5))
+  (segment (start 147.95 124) (end 149.49 122.46) (width 0.5) (layer B.Cu) (net 5))
+  (segment (start 146 124) (end 147.95 124) (width 0.5) (layer B.Cu) (net 5))
+  (segment (start 152.5 100.265998) (end 152.969002 100.265998) (width 0.5) (layer B.Cu) (net 6))
+  (segment (start 151.469999 101.295999) (end 152.5 100.265998) (width 0.5) (layer B.Cu) (net 6))
+  (segment (start 151.469999 102.757) (end 151.469999 101.295999) (width 0.5) (layer B.Cu) (net 6))
+  (segment (start 152.969002 100.265998) (end 154.155 99.08) (width 0.5) (layer B.Cu) (net 6))
+  (segment (start 152.5 103.787001) (end 151.469999 102.757) (width 0.5) (layer B.Cu) (net 6))
+  (segment (start 152.5 116.655) (end 152.5 103.787001) (width 0.5) (layer B.Cu) (net 6))
+  (segment (start 148.475 120.68) (end 152.5 116.655) (width 0.5) (layer B.Cu) (net 6))
+  (segment (start 150.535001 99.929999) (end 151.385 99.08) (width 0.5) (layer B.Cu) (net 7))
+  (segment (start 150.065999 99.929999) (end 150.535001 99.929999) (width 0.5) (layer B.Cu) (net 7))
+  (segment (start 148.699999 101.295999) (end 150.065999 99.929999) (width 0.5) (layer B.Cu) (net 7))
+  (segment (start 148.699999 104.800001) (end 148.699999 101.295999) (width 0.5) (layer B.Cu) (net 7))
+  (segment (start 147.5 106) (end 148.699999 104.800001) (width 0.5) (layer B.Cu) (net 7))
+  (segment (start 147.5 119.625) (end 147.5 106) (width 0.5) (layer B.Cu) (net 7))
+  (segment (start 146.445 120.68) (end 147.5 119.625) (width 0.5) (layer B.Cu) (net 7))
+  (segment (start 145.845 109.955) (end 145.3 110.5) (width 0.5) (layer F.Cu) (net 9))
+  (segment (start 145.845 99.08) (end 145.845 109.955) (width 0.5) (layer F.Cu) (net 9))
+  (segment (start 146.39934 122.46) (end 147.46 122.46) (width 0.5) (layer B.Cu) (net 9))
+  (segment (start 145 121.06066) (end 146.39934 122.46) (width 0.5) (layer B.Cu) (net 9))
+  (segment (start 145 112.92132) (end 145 121.06066) (width 0.5) (layer B.Cu) (net 9))
+  (segment (start 145.3 112.62132) (end 145 112.92132) (width 0.5) (layer B.Cu) (net 9))
+  (segment (start 145.3 110.5) (end 145.3 112.62132) (width 0.5) (layer B.Cu) (net 9))
+  (segment (start 154.7 118.515) (end 154.7 110.5) (width 0.5) (layer B.Cu) (net 10))
+  (segment (start 152.535 120.68) (end 154.7 118.515) (width 0.5) (layer B.Cu) (net 10))
   (zone (net 8) (net_name /GND) (layer F.Cu) (hatch edge 0.508)
     (connect_pads (clearance 0.508))

Commit message: updated bottom silk
Parts:
- added G***: LOGO, logos:gmlogo, B.Cu at (150.0, 116.5)
Other:
- board text added: "C64 / Amiga"
- board text removed: "good micros"
